File: devices/kicad/kicad_project.kicad_pcb (KiCad board)
At the start: 2 copper layers, 8 parts, among them U1 SIM800L, U2 esp32_NodeMCU-track_chip, U3 GPS_PA6H, U4 bmp180-track_chip, U5 polulu, U7 charger_mr010

Commit message: [PCB] Premier jet
Parts:
- removed D2: D, Diode_THT:D_DO-15_P10.16mm_Horizontal
- added D1: 0.8V, Diode_THT:D_DO-15_P10.16mm_Horizontal, F.Cu at (202.6, 128.3)
- C1: value C -> 100u
- moved C1 75.7 mm to (214.5, 101.7), turned to 0 degrees
- moved U7 75.0 mm to (144.4, 117.1)
- moved U4 68.1 mm to (212.8, 78.9)
- moved U5 59.9 mm to (169.0, 124.0), turned to 90 degrees
- moved U2 59.5 mm to (104.8, 78.2)
- moved U1 46.1 mm to (211.1, 111.4)
- moved U3 41.6 mm to (167.9, 73.3)
Connections:
- net Net-(U2-Pad16) renamed 3V3
- U1 pad 4: RX0 -> RX2
- U1 pad 5: TX0 -> TX2
- U2 pad 15: Net-(U2-Pad15) -> VBAT
- U2 pad 20: Net-(U2-Pad20) -> EN_GPS
- U3 pad 2: Net-(U3-Pad2) -> EN_GPS
- U5 pad 4: 5V -> Net-(D1-Pad2)
Routing:
- net VBAT: track 0.00 -> 107.4 mm
- net SCL: track 0.00 -> 103.5 mm
- net SDA: track 0.00 -> 95.3 mm
- net TX2: track 0.00 -> 90.3 mm
- net RX2: track 0.00 -> 88.1 mm
- net GND: track 0.00 -> 81.5 mm
- net RX0: track 0.00 -> 37.5 mm
- net TX0: track 0.00 -> 37.4 mm
- net Net-(C1-Pad1): track 0.00 -> 23.6 mm
- net Net-(D1-Pad2): track 0.00 -> 18.5 mm
