File: devices/kicad/version_sim/kicad_project.kicad_pcb (KiCad board)
At the start: 2 copper layers, 8 parts, among them U1 SIM800L, U2 esp32_NodeMCU-track_chip, U3 GPS_PA6H, U4 bmp180-track_chip, U5 polulu, U7 charger_mr010

Commit message: [PCB] version sim en cours
Parts:
- moved U4 101.7 mm to (112.6, 61.4), turned to 90 degrees
Routing:
- net GND: track 81.5 -> 0.52 mm
- net SCL: track 103.5 -> 35.0 mm
- net SDA: track 95.3 -> 33.3 mm
Changed lines of the file:
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@@
     (thickness 1.6)
     (drawings 0)
-    (tracks 69)
+    (tracks 57)
     (zones 0)
     (modules 8)
@@
   )
   (module track_chip:bmp180 (layer F.Cu)
-    (at 212.8012 78.8924)
-    (fp_text reference U4 (at 8.89 -1.905) (layer F.SilkS)
-      (effects (font (size 1 1) (thickness 0.15)))
-    )
-    (fp_text value bmp180-track_chip (at 8.255 0) (layer F.Fab)
+    (at 112.5728 61.4172 90)
+    (fp_text reference U4 (at 8.89 -1.905 90) (layer F.SilkS)
+      (effects (font (size 1 1) (thickness 0.15)))
+    )
+    (fp_text value bmp180-track_chip (at 8.255 0 90) (layer F.Fab)
       (effects (font (size 1 1) (thickness 0.15)))
     )
@@
     (fp_line (start 19.05 -4.445) (end -1.27 -4.445) (layer F.SilkS) (width 0.12))
     (fp_line (start -1.27 -4.445) (end -1.27 10.16) (layer F.SilkS) (width 0.12))
-    (pad 1 thru_hole rect (at 0 0) (size 1.524 1.524) (drill 0.762) (layers *.Cu *.Mask)
+    (pad 1 thru_hole rect (at 0 0 90) (size 1.524 1.524) (drill 0.762) (layers *.Cu *.Mask)
       (net 11 3.3V))
-    (pad 2 thru_hole circle (at 0 2.54) (size 1.524 1.524) (drill 0.762) (layers *.Cu *.Mask)
+    (pad 2 thru_hole circle (at 0 2.54 90) (size 1.524 1.524) (drill 0.762) (layers *.Cu *.Mask)
       (net 11 3.3V))
-    (pad 3 thru_hole circle (at 0 5.08) (size 1.524 1.524) (drill 0.762) (layers *.Cu *.Mask)
-      (net 6 GND))
-    (pad 4 thru_hole circle (at 0 7.62) (size 1.524 1.524) (drill 0.762) (layers *.Cu *.Mask)
+    (pad 3 thru_hole circle (at 0 5.08 90) (size 1.524 1.524) (drill 0.762) (layers *.Cu *.Mask)
+      (net 6 GND))
+    (pad 4 thru_hole circle (at 0 7.62 90) (size 1.524 1.524) (drill 0.762) (layers *.Cu *.Mask)
       (net 36 SCL))
-    (pad 5 thru_hole circle (at 0 10.16) (size 1.524 1.524) (drill 0.762) (layers *.Cu *.Mask)
+    (pad 5 thru_hole circle (at 0 10.16 90) (size 1.524 1.524) (drill 0.762) (layers *.Cu *.Mask)
       (net 34 SDA))
   )
@@
   (segment (start 130.2004 85.852) (end 167.6908 85.852) (width 1) (layer B.Cu) (net 4))
   (segment (start 130.2004 83.312) (end 167.64 83.312) (width 1) (layer B.Cu) (net 5))
-  (segment (start 209.3468 82.9056) (end 210.5152 84.074) (width 1) (layer B.Cu) (net 6))
-  (segment (start 209.3468 71.9836) (end 209.3468 82.9056) (width 1) (layer B.Cu) (net 6))
-  (segment (start 210.5152 84.074) (end 212.598 84.074) (width 1) (layer B.Cu) (net 6))
-  (segment (start 239.6744 76.1492) (end 232.6132 69.088) (width 1) (layer B.Cu) (net 6))
-  (segment (start 232.6132 69.088) (end 212.2424 69.088) (width 1) (layer B.Cu) (net 6))
-  (segment (start 212.2424 69.088) (end 209.3468 71.9836) (width 1) (layer B.Cu) (net 6))
-  (segment (start 239.6744 76.1492) (end 239.6744 95.4024) (width 1) (layer B.Cu) (net 6))
-  (segment (start 239.6744 95.4024) (end 233.4768 101.6) (width 1) (layer B.Cu) (net 6))
-  (segment (start 233.4768 101.6) (end 229.6668 101.6) (width 1) (layer B.Cu) (net 6))
   (segment (start 229.6668 101.6) (end 229.5144 101.4476) (width 1) (layer B.Cu) (net 6))
   (segment (start 229.5144 101.4476) (end 229.5144 101.7524) (width 1) (layer B.Cu) (net 6))
@@
   (segment (start 130.2004 98.552) (end 146.6596 98.552) (width 1) (layer B.Cu) (net 30))
   (segment (start 146.6596 98.552) (end 152.0952 103.9876) (width 1) (layer B.Cu) (net 30))
-  (segment (start 130.2004 88.392) (end 143.9672 88.392) (width 1) (layer B.Cu) (net 34))
-  (segment (start 143.9672 88.392) (end 155.5496 99.9744) (width 1) (layer B.Cu) (net 34))
-  (segment (start 155.5496 99.9744) (end 203.6572 99.9744) (width 1) (layer B.Cu) (net 34))
-  (segment (start 203.6572 99.9744) (end 205.5368 98.0948) (width 1) (layer B.Cu) (net 34))
-  (segment (start 205.5368 98.0948) (end 205.5368 91.9988) (width 1) (layer B.Cu) (net 34))
-  (segment (start 205.5368 91.9988) (end 208.3816 89.154) (width 1) (layer B.Cu) (net 34))
-  (segment (start 208.3816 89.154) (end 212.6488 89.154) (width 1) (layer B.Cu) (net 34))
-  (segment (start 130.962399 80.010001) (end 141.884399 80.010001) (width 1) (layer B.Cu) (net 36))
+  (segment (start 122.7328 61.4172) (end 122.7328 86.1568) (width 1) (layer B.Cu) (net 34))
+  (segment (start 122.7328 86.1568) (end 125.2728 88.6968) (width 1) (layer B.Cu) (net 34))
+  (segment (start 125.2728 88.6968) (end 130.2512 88.6968) (width 1) (layer B.Cu) (net 34))
   (segment (start 130.2004 80.772) (end 130.962399 80.010001) (width 1) (layer B.Cu) (net 36))
-  (segment (start 141.884399 80.010001) (end 154.94 66.9544) (width 1) (layer B.Cu) (net 36))
-  (segment (start 154.94 66.9544) (end 202.1332 66.9544) (width 1) (layer B.Cu) (net 36))
-  (segment (start 202.1332 66.9544) (end 207.0608 71.882) (width 1) (layer B.Cu) (net 36))
-  (segment (start 207.0608 71.882) (end 207.0608 84.328) (width 1) (layer B.Cu) (net 36))
-  (segment (start 207.0608 84.328) (end 209.3468 86.614) (width 1) (layer B.Cu) (net 36))
-  (segment (start 209.3468 86.614) (end 212.5472 86.614) (width 1) (layer B.Cu) (net 36))
+  (segment (start 119.430801 60.655201) (end 119.430801 59.588399) (width 1) (layer B.Cu) (net 36))
+  (segment (start 120.1928 61.4172) (end 119.430801 60.655201) (width 1) (layer B.Cu) (net 36))
+  (segment (start 119.430801 59.588399) (end 120.7008 58.3184) (width 1) (layer B.Cu) (net 36))
+  (segment (start 120.7008 58.3184) (end 123.9012 58.3184) (width 1) (layer B.Cu) (net 36))
+  (segment (start 123.9012 58.3184) (end 125.8824 60.2996) (width 1) (layer B.Cu) (net 36))
+  (segment (start 125.8824 60.2996) (end 125.8824 79.9084) (width 1) (layer B.Cu) (net 36))
+  (segment (start 125.8824 79.9084) (end 126.8476 80.8736) (width 1) (layer B.Cu) (net 36))
+  (segment (start 126.8476 80.8736) (end 129.8956 80.8736) (width 1) (layer B.Cu) (net 36))
   (segment (start 176.6316 125.08043) (end 180.02437 128.4732) (width 1) (layer B.Cu) (net 38))
   (segment (start 176.6316 124.0028) (end 176.6316 125.08043) (width 1) (layer B.Cu) (net 38))
