File: devices/kicad/version_gsm/kicad_project.kicad_pcb (KiCad board)
At the start: 2 copper layers, 8 parts, among them U1 SIM800L, U2 esp32_NodeMCU-track_chip, U3 GPS_PA6H, U4 bmp180-track_chip, U5 polulu, U7 charger_mr010

Commit message: [PCB] Premier jet GSM
Parts:
- added G***: LOGO, track_chip:logo, F.Cu at (100.1, 91.4)
- moved U1 67.6 mm to (144.1, 102.5), turned to 270 degrees
- moved U7 53.6 mm to (193.4, 95.4), turned to 180 degrees
- moved U3 38.9 mm to (157.6, 110.8), turned to 90 degrees
- moved U4 33.6 mm to (142.4, 76.8), turned to 270 degrees
- moved C1 25.5 mm to (190.2, 109.6), turned to 270 degrees
- moved D1 24.0 mm to (183.4, 113.8), turned to 270 degrees
- moved U2 9.97 mm to (95.4, 81.6)
- moved U5 4.22 mm to (173.0, 125.3), turned to 180 degrees
Connections:
- D1 pad 2: Net-(D1-Pad2) -> 5V
- U1 pad 1: Net-(U1-Pad1) -> (no net)
- U1 pad 3: Net-(U1-Pad3) -> (no net)
- U2 pad 1: Net-(U2-Pad1) -> (no net)
- U2 pad 10: Net-(U2-Pad10) -> (no net)
- U2 pad 11: Net-(U2-Pad11) -> (no net)
- U2 pad 12: Net-(U2-Pad12) -> (no net)
- U2 pad 13: Net-(U2-Pad13) -> (no net)
- U2 pad 14: Net-(U2-Pad14) -> (no net)
- U2 pad 15: VBAT -> 5V
- U2 pad 16: 3V3 -> (no net)
- U2 pad 18: Net-(U2-Pad18) -> (no net)
- U2 pad 19: Net-(U2-Pad19) -> (no net)
- U2 pad 2: Net-(U2-Pad2) -> (no net)
- U2 pad 20: EN_GPS -> (no net)
- U2 pad 23: Net-(U2-Pad23) -> (no net)
- U2 pad 24: Net-(U2-Pad24) -> EN_GPS
- U2 pad 25: Net-(U2-Pad25) -> (no net)
- U2 pad 27: RX0 -> (no net)
- U2 pad 3: Net-(U2-Pad3) -> (no net)
- U2 pad 30: Net-(U2-Pad30) -> (no net)
- U2 pad 4: Net-(U2-Pad4) -> (no net)
- U2 pad 5: Net-(U2-Pad5) -> (no net)
- U2 pad 6: Net-(U2-Pad6) -> (no net)
- U2 pad 7: Net-(U2-Pad7) -> (no net)
- U2 pad 8: Net-(U2-Pad8) -> (no net)
- U2 pad 9: Net-(U2-Pad9) -> (no net)
- U3 pad 1: Net-(U3-Pad1) -> (no net)
- U3 pad 3: Net-(U3-Pad3) -> (no net)
- U3 pad 4: Net-(U3-Pad4) -> (no net)
- U3 pad 6: RX0 -> (no net)
- U3 pad 9: Net-(U3-Pad9) -> (no net)
- U5 pad 1: Net-(U5-Pad1) -> (no net)
- U5 pad 4: Net-(D1-Pad2) -> 5V
Routing:
- net 5V: track 0.00 -> 115.3 mm
- net TX2: track 90.3 -> 19.5 mm
- net RX2: track 88.1 -> 24.6 mm
- net 3.3V: track 0.00 -> 62.1 mm
- net VBAT: track 107.4 -> 45.8 mm
- net EN_GPS: track 0.00 -> 54.7 mm
- net RX0: track 37.5 -> 0.00 mm
- net Net-(C1-Pad1): track 23.6 -> 58.7 mm
- net TX0: track 37.4 -> 59.2 mm
- net Net-(D1-Pad2): track 18.5 -> 0.00 mm
- net SCL: track 35.0 -> 21.6 mm
- net SDA: track 33.3 -> 32.2 mm
- net GND: track 0.52 -> 0.00 mm
